File: h-bridge-driver/h-bridge-driver.kicad_pcb (KiCad board)
At the start: 2 copper layers, 0 parts

Commit message: Complete H bridge driver
Parts:
- added C1: CAP_CER_100NF_25V_0402, connaxio-capacitors:CAP_CER_0402_1005M, F.Cu at (119.5, 50.6)
- added C2: CAP_AE_22UF_100V_TH_6.3MM, connaxio-capacitors:CAP_AE_RAD_D6.3_H12.5_P2.5, F.Cu at (117.5, 85.3)
- added C3: CAP_CER_100NF_25V_0402, connaxio-capacitors:CAP_CER_0402_1005M, F.Cu at (121.8, 51.9)
- added C4: CAP_CER_100NF_25V_0402, connaxio-capacitors:CAP_CER_0402_1005M, F.Cu at (122.2, 58.2)
- added C5: CAP_CER_100NF_25V_0402, connaxio-capacitors:CAP_CER_0402_1005M, F.Cu at (116.2, 57.4)
- added C6: CAP_CER_100NF_25V_0402, connaxio-capacitors:CAP_CER_0402_1005M, F.Cu at (118.5, 57.4)
- added C7: CAP_CER_1UF_25V_0603, connaxio-capacitors:CAP_CER_0603_1608M, F.Cu at (116.8, 50.4)
- added C8: CAP_CER_10UF_25V_1206, connaxio-capacitors:CAP_CER_1206_3216M, F.Cu at (122.1, 55.1)
- added J1: CON_HDR_100MILS_M_TH_2X8, connaxio-connectors:CON_HDR_100MILS_M_TH_2X8, B.Cu at (116.5, 71.1)
- added J2: CON_TERM_BLK_1X2_TB008A-508-02BE, connaxio-connectors:CON_TERM_BLK_1X2_TB008A-508-02BE, F.Cu at (131.1, 68.6)
- added Q1: TRX_NMOS_PJD40N04_L2_00001, connaxio-sop:TO-252-3, F.Cu at (135.6, 80.1)
- added Q2: TRX_NMOS_PJD40N04_L2_00001, connaxio-sop:TO-252-3, F.Cu at (128.5, 80.1)
- added Q3: TRX_NMOS_PJD40N04_L2_00001, connaxio-sop:TO-252-3, F.Cu at (135.6, 56.9)
- added Q4: TRX_NMOS_PJD40N04_L2_00001, connaxio-sop:TO-252-3, F.Cu at (128.4, 56.9)
- added R1: RES_5.10KΩ_1%_0402, connaxio-resistors:RES_0402_1005M, F.Cu at (120.7, 66.1)
- added R2: RES_5.10KΩ_1%_0402, connaxio-resistors:RES_0402_1005M, F.Cu at (120.8, 68.7)
- added R3: RES_226Ω_1%_0402, connaxio-resistors:RES_0402_1005M, F.Cu at (121.2, 71.0)
- added R4: RES_5.10KΩ_1%_0402, connaxio-resistors:RES_0402_1005M, F.Cu at (118.5, 58.8)
- added R5: RES_226Ω_1%_0402, connaxio-resistors:RES_0402_1005M, F.Cu at (121.9, 50.5)
- added R6: RES_226Ω_1%_0402, connaxio-resistors:RES_0402_1005M, F.Cu at (122.5, 61.9)
- added R7: RES_226Ω_1%_0402, connaxio-resistors:RES_0402_1005M, F.Cu at (119.8, 71.0)
- added U1: DRV_A4957SESTR-T, connaxio-fp:QFN-24_4x4_P0.5_EP2.7X2.7, F.Cu at (117.8, 54.0)
Routing:
- net Vdrive: track 0.00 -> 56.0 mm, vias 0 -> 29
- net /OUTA: track 0.00 -> 30.0 mm
- net Net-(Q1-Pad1): track 0.00 -> 23.0 mm, vias 0 -> 2
- net +3.3V: track 0.00 -> 22.5 mm
- net GND: track 0.00 -> 21.0 mm, vias 0 -> 49
- net Net-(U1-Pad24): track 0.00 -> 20.0 mm, vias 0 -> 2
- net Net-(Q3-Pad1): track 0.00 -> 19.1 mm
- net /FAULT: track 0.00 -> 18.9 mm, vias 0 -> 2
- net /RST: track 0.00 -> 18.2 mm, vias 0 -> 1
- net Net-(U1-Pad20): track 0.00 -> 17.5 mm, vias 0 -> 2
- net Net-(Q2-Pad1): track 0.00 -> 16.2 mm, vias 0 -> 2
- net /OUTB: track 0.00 -> 15.6 mm
- net /CTRLB: track 0.00 -> 13.3 mm, vias 0 -> 1
- net /CTRLA: track 0.00 -> 12.7 mm
- net Net-(U1-Pad18): track 0.00 -> 7.24 mm
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- added copper zone on F.Cu, net /OUTA
- added copper zone on F.Cu, net /OUTB
- added copper zone on B.Cu, net GND
- added copper zone on F.Cu, net GND
- added copper zone on In1.Cu, net GND
- added copper zone on In2.Cu, net GND
- added copper zone on B.Cu, net Vdrive
- added copper zone on F.Cu, net Vdrive
- added copper zone on In1.Cu, net Vdrive
- added copper zone on In2.Cu, net Vdrive
Other:
- board outline added: 25.4 x 40.6 mm
- copper layers 2 -> 4
- rule pad_to_mask_clearance: 0.0508 -> 0.05
- rule solder_mask_min_width: 0.0508 -> 0.05
