File: h-bridge-driver/h-bridge-driver.kicad_sch (KiCad schematic)
At the start: 37 parts, among them J1 CON_HDR_100MILS_M_TH_2X8, J2 CON_HDR_100MILS_M_TH_1X3, J3 CON_TERM_BLK_1X2_TB008A-508-0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, Q1 TRX_2NPN_BC846S,115, Q2 TRX_NMOS_PJD40N04_L2_00001, Q3 TRX_NMOS_PJD40N04_L2_00001, Q4 TRX_NMOS_PJD40N04_L2_00001, Q5 TRX_NMOS_PJD40N04_L2_00001, U1 DRV_A4957SESTR-T

Commit message: Invert connectors (male/female) Replace TH connectors with SMD ones on mainboard Add 555 timer on simple-switch to generate 60 Hz Add jumper on simple-switch to select AC Add series I2C resistors on mainboard from mikroBUS socket
Parts:
- removed J1: CON_HDR_100MILS_M_TH_2X8, connaxio-connectors:CON_HDR_100MILS_M_TH_2X8, symbol connaxio-connectors:CON_HDR_100MILS_M_TH_2X8
- added J1: CON_HDR_100MILS_F_TH_2X8, connaxio-connectors:CON_HDR_100MILS_F_TH_2X8, symbol connaxio-connectors:CON_HDR_100MILS_F_TH_2X8
Connections:
- net +3.3V: now also J1.5
- net GND: now also J1.10, J1.12, J1.7, J1.8, J1.9
- net VIN: now also J1.11, J1.13, J1.14, J1.15, J1.16
- net ~{CTRLA}: now also J1.1
- net ~{CTRLB}: now also J1.3
- net ~{FAULT}: now also J1.2
- net ~{RST}: now also J1.4
