File: mainboard/greenhouse_controller_makroshield.kicad_pcb (KiCad board)
At the start: 2 copper layers, 0 parts

Commit message: Move fuse to motor driver board Optimize board array schematic (hierarchical schematics)
Parts:
- added C1: CAP_AE_1MF_50V_TH_12.5MM, connaxio-capacitors:CAPAE_RAD_D12.5_H26.5_P5, F.Cu at (30.3, 60.7)
- added C2: CAP_CER_100NF_25V_0402, connaxio-capacitors:CAP_CER_0402_1005M, F.Cu at (94.5, 34.5)
- added C3: CAP_CER_100NF_25V_0402, connaxio-capacitors:CAP_CER_0402_1005M, F.Cu at (85.4, 43.6)
- added C4: CAP_CER_100NF_25V_0402, connaxio-capacitors:CAP_CER_0402_1005M, F.Cu at (65.9, 65.0)
- added C5: CAP_CER_22UF_10V_0603, connaxio-capacitors:CAP_CER_0603_1608M, F.Cu at (97.5, 25.6)
- added C6: CAP_CER_100NF_25V_0402, connaxio-capacitors:CAP_CER_0402_1005M, F.Cu at (80.9, 47.2)
- added C7: CAP_CER_10UF_25V_1206, connaxio-capacitors:CAP_CER_1206_3216M, F.Cu at (82.2, 39.8)
- added C8: CAP_CER_100NF_25V_0402, connaxio-capacitors:CAP_CER_0402_1005M, F.Cu at (80.9, 49.5)
- added D1: DIO_TVS_24V_UNI_SMB, connaxio-diodes:DO-124AA_SMB, F.Cu at (61.9, 49.4)
- added D2: DIO_TVS_24V_UNI_SMB, connaxio-diodes:DO-124AA_SMB, F.Cu at (49.8, 64.6)
- added D3: DIO_SBD_100V_3A_SMA, connaxio-diodes:DO-214AC_SMA, F.Cu at (82.2, 35.8)
- added D4: DIO_TVS_5V_UNI_SMA, connaxio-diodes:DO-214AC_SMA, F.Cu at (93.2, 20.3)
- added F1: FUS_BLADE_3522, connaxio-connectors:FUS_BLADE_3522, F.Cu at (60.8, 43.5)
- added F2: FID_1X3, connaxio-mechanical:FID_1X3, F.Cu at (68.3, 48.9)
- added F3: FID_1X3, connaxio-mechanical:FID_1X3, F.Cu at (105.8, 20.3)
- added F4: FID_1X3, connaxio-mechanical:FID_1X3, F.Cu at (81.6, 43.8)
- added F5: FID_1X3, connaxio-mechanical:FID_1X3, F.Cu at (91.5, 31.1)
- added J1: CON_TERM_BLK_1X2_TB008A-508-02BE, connaxio-connectors:CON_TERM_BLK_1X2_TB008A-508-02BE, F.Cu at (52.0, 53.3)
- added J10: CON_CONNAXIO_MOTOR_DRIVER, connaxio-connectors:CON_CONNAXIO_MOTOR_DRIVER, F.Cu at (33.9, 179.1)
- added J11: CON_CONNAXIO_MOTOR_DRIVER, connaxio-connectors:CON_CONNAXIO_MOTOR_DRIVER, F.Cu at (107.6, 118.1)
- added J12: CON_CONNAXIO_MOTOR_DRIVER, connaxio-connectors:CON_CONNAXIO_MOTOR_DRIVER, F.Cu at (107.6, 148.6)
- added J13: CON_CONNAXIO_MOTOR_DRIVER, connaxio-connectors:CON_CONNAXIO_MOTOR_DRIVER, F.Cu at (144.4, 148.6)
- added J14: CON_CONNAXIO_MOTOR_DRIVER, connaxio-connectors:CON_CONNAXIO_MOTOR_DRIVER, F.Cu at (144.4, 118.1)
- added J15: CON_CONNAXIO_MOTOR_DRIVER, connaxio-connectors:CON_CONNAXIO_MOTOR_DRIVER, F.Cu at (144.4, 179.1)
- added J16: CON_CONNAXIO_MOTOR_DRIVER, connaxio-connectors:CON_CONNAXIO_MOTOR_DRIVER, F.Cu at (33.9, 87.6)
- added J17: CON_CONNAXIO_MOTOR_DRIVER, connaxio-connectors:CON_CONNAXIO_MOTOR_DRIVER, F.Cu at (70.7, 87.6)
- added J18: CON_CONNAXIO_MOTOR_DRIVER, connaxio-connectors:CON_CONNAXIO_MOTOR_DRIVER, F.Cu at (70.7, 179.1)
- added J19: CON_CONNAXIO_MOTOR_DRIVER, connaxio-connectors:CON_CONNAXIO_MOTOR_DRIVER, F.Cu at (107.6, 87.6)
- added J2: CON_HDR_MIKROBUS_ADDON_TH, connaxio-connectors:CON_HDR_MIKROBUS_ADDON_TH, B.Cu at (177.4, 146.1)
- added J3: CON_HDR_MIKROBUS_SOCKET_TH, connaxio-connectors:CON_HDR_MIKROBUS_SOCKET_TH, F.Cu at (36.9, 33.1)
- added J4: CON_CONNAXIO_MOTOR_DRIVER, connaxio-connectors:CON_CONNAXIO_MOTOR_DRIVER, F.Cu at (70.7, 118.1)
- added J5: CON_CONNAXIO_MOTOR_DRIVER, connaxio-connectors:CON_CONNAXIO_MOTOR_DRIVER, F.Cu at (107.6, 179.1)
- added J6: CON_CONNAXIO_MOTOR_DRIVER, connaxio-connectors:CON_CONNAXIO_MOTOR_DRIVER, F.Cu at (33.9, 118.1)
- added J7: CON_CONNAXIO_MOTOR_DRIVER, connaxio-connectors:CON_CONNAXIO_MOTOR_DRIVER, F.Cu at (144.4, 87.6)
- added J8: CON_CONNAXIO_MOTOR_DRIVER, connaxio-connectors:CON_CONNAXIO_MOTOR_DRIVER, F.Cu at (70.7, 148.6)
- added J9: CON_CONNAXIO_MOTOR_DRIVER, connaxio-connectors:CON_CONNAXIO_MOTOR_DRIVER, F.Cu at (33.9, 148.6)
- added MTH1: MTH_M2.5_PTH_CORNER, connaxio-mechanical:MTH_M2.5_PTH_CORNER, F.Cu at (61.0, 55.6)
- added MTH2: MTH_M2.5_NPTH, connaxio-mechanical:MTH_M2.5_NPTH, F.Cu at (89.6, 36.9)
- added MTH3: MTH_M2.5_NPTH, connaxio-mechanical:MTH_M2.5_NPTH, F.Cu at (69.4, 55.2)
- added MTH4: MTH_M2.5_NPTH, connaxio-mechanical:MTH_M2.5_NPTH, F.Cu at (61.0, 62.3)
- added Q1: TRX_PMOS_AOD4189, connaxio-sop:TO-252-3, F.Cu at (41.5, 59.9)
- added Q2: TRX_NPN_MMBT3904-TP, connaxio-sop:SOT-23-3, F.Cu at (96.0, 31.1)
- added R1: NTC_SL22 2R018, connaxio-resistors:RV_DISC_D22_W6_P7.8, F.Cu at (34.7, 49.9)
- added R10: RES_12.4KΩ_1%_0402, connaxio-resistors:RES_0402_1005M, F.Cu at (105.1, 23.6)
- added R11: RES_1.54KΩ_1%_0402, connaxio-resistors:RES_0402_1005M, F.Cu at (55.5, 65.2)
- added R12: RES_12.4KΩ_1%_0402, connaxio-resistors:RES_0402_1005M, F.Cu at (101.2, 25.4)
- added R13: RES_0Ω_0402, connaxio-resistors:RES_0402_1005M, F.Cu at (61.9, 66.8)
- added R14: RES_12.4KΩ_1%_0402, connaxio-resistors:RES_0402_1005M, F.Cu at (55.5, 63.0)
- added R2: RES_12.4KΩ_1%_0402, connaxio-resistors:RES_0402_1005M, F.Cu at (101.2, 27.6)
- added R3: RES_12.4KΩ_1%_0402, connaxio-resistors:RES_0402_1005M, F.Cu at (42.2, 67.3)
- added R4: RES_12.4KΩ_1%_0402, connaxio-resistors:RES_0402_1005M, F.Cu at (74.4, 53.0)
- added R5: RES_1.54KΩ_1%_0402, connaxio-resistors:RES_0402_1005M, F.Cu at (55.5, 67.4)
- added R6: RES_1.54KΩ_1%_0402, connaxio-resistors:RES_0402_1005M, F.Cu at (58.7, 66.8)
- added R7: RES_12.4KΩ_1%_0402, connaxio-resistors:RES_0402_1005M, F.Cu at (109.7, 19.1)
- added R8: RES_226Ω_1%_0402, connaxio-resistors:RES_0402_1005M, F.Cu at (39.1, 67.3)
- added R9: RES_226Ω_1%_0402, connaxio-resistors:RES_0402_1005M, F.Cu at (86.7, 41.4)
- added U1: IO_EXP_PI4IOE5V6416ZDEX, connaxio-fp:QFN-24_4x4_P0.5_EP2.7X2.7, F.Cu at (92.3, 25.7)
- added U2: IO_EXP_PI4IOE5V6416ZDEX, connaxio-fp:QFN-24_4x4_P0.5_EP2.7X2.7, F.Cu at (100.4, 21.1)
- added U3: CON_BARREL_2.1X5.5_PJ-002A, connaxio-connectors:CON_BARREL_2.1X5.5_PJ-002A, F.Cu at (83.2, 25.8)
- added U4: SUN_CUR_ACS711KEXLT-31AB-T, connaxio-fp:QFN-12_CUR_SEN_ACS7, F.Cu at (67.0, 61.2)
- added U5: ADC_NAU7802SGI, connaxio-sop:SOIC-16_3.9X9.9_P1.27, F.Cu at (75.1, 46.1)
Other:
- board outline added: 175.3 x 177.8 mm
